File: 00-produccion-pcbs/1-versiones-profes/grupo-05/g-05-filt-01-rev-a/g-05-filt-01-rev-a.kicad_pcb (KiCad board)
At the start: 2 copper layers, 106.7 x 97.3 mm, 14 parts, among them J4 AudioJack2_SwitchT, J5 AudioJack2_SwitchT

Commit message: añadido g05
Parts:
- C1: value 1uf -> 1u; footprint Capacitor_THT:CP_Radial_D5.0mm_P2.00mm -> Capacitor_THT:C_Disc_D10.5mm_W5.0mm_P7.50mm
- C4: value 153n -> 15n
- C5: value 154n -> 150n
- moved C1 16.3 mm to (116.3, 98.7), turned to 45 degrees
- renumbered J5 to J1, J4 to J2
Connections:
- C4 pad 1: Net-(C1-Pad1) -> Net-(C1-Pad2)
- C5 pad 2: Net-(C1-Pad2) -> Net-(C1-Pad1)
- J1 pad 3: Net-(C1-Pad2) -> Net-(C1-Pad1)
- J2 pad 3: Net-(C1-Pad2) -> Net-(C1-Pad1)
- R1 pad 1: Net-(C1-Pad1) -> Net-(C1-Pad2)
- R2 pad 2: Net-(C1-Pad2) -> Net-(C1-Pad1)
- R3 pad 2: Net-(C1-Pad2) -> Net-(C1-Pad1)
- RV1 pad 2: unconnected-(RV1-Pad2) -> Net-(C2-Pad2)
- RV2 pad 2: unconnected-(RV2-Pad2) -> Net-(C1-Pad1)
Routing:
- net Net-(C1-Pad1): track 59.7 -> 210.7 mm, vias 0 -> 1
- net Net-(C2-Pad2): track 58.4 -> 118.6 mm
- net Net-(C1-Pad2): track 241.6 -> 187.0 mm, vias 0 -> 2
- added copper zone on B.Cu, net GND
- added copper zone on F.Cu, net GND
Other:
- board text added: "g-05-filt-01-rev-a"
