File: 00-produccion-pcbs/1-versiones-profes/grupo-05/g-05-filt-01-rev-a/g-05-filt-01-rev-a.kicad_sch (KiCad schematic)
At the start: 14 parts, among them J4 AudioJack2_SwitchT, J5 AudioJack2_SwitchT

Commit message: añadido g05
Parts:
- removed C1: 1uf, Capacitor_THT:CP_Radial_D5.0mm_P2.00mm, symbol Device:C_Polarized
- removed R4: 10k, Resistor_THT:R_Axial_DIN0207_L6.3mm_D2.5mm_P2.54mm_Vertical, symbol Device:R
- removed R5: 1k, Resistor_THT:R_Axial_DIN0207_L6.3mm_D2.5mm_P2.54mm_Vertical, symbol Device:R
- added C1: 1u, Capacitor_THT:C_Disc_D10.5mm_W5.0mm_P7.50mm, symbol Device:C
- C4: value 153n -> 15n
- C5: value 154n -> 150n
- renumbered J5 to J1, J4 to J2
Connections:
- net at RV1.2: now also C2.2, C3.2, R3.1
- net at C5.2, J1.3, J2.3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: now also RV2.2, C1.1
- net at C4.1, R1.1: now also C1.2
Other:
- note added: "basado en https://www.homemade-circuits.com/simple-tone-control-circuits/"
- moved on the sheet: RV1, RV2
