File: 00-produccion-pcbs/1-versiones-profes/grupo-06/g-06-perc-01-rev-a/g-06-perc-01-rev-a.kicad_pcb (KiCad board)
At the start: 2 copper layers, 98.5 x 99.4 mm, 29 parts, among them J2 Barrel_Jack_Switch, J3 Barrel_Jack_Switch, J4 AudioJack2_SwitchT, SW3 SW_SPDT, U2 40106, U3 4069, U8 L7805

Commit message: añadido g06-01
Parts:
- added J5: AudioJack2_SwitchT, dis8644:PJ301M-12, F.Cu at (149.3, 127.4)
Connections:
- U2 pad 1: Net-(C14-Pad1) -> Net-(J5-Pad3)
- U2 pad 11: unconnected-(U2-Pad11) -> GND
- U2 pad 13: unconnected-(U2-Pad13) -> GND
- U2 pad 5: unconnected-(U2-Pad5) -> GND
- U2 pad 9: unconnected-(U2-Pad9) -> GND
- U3 pad 11: unconnected-(U3-Pad11) -> GND
- U3 pad 13: unconnected-(U3-Pad13) -> GND
- U3 pad 5: unconnected-(U3-Pad5) -> GND
- U3 pad 9: unconnected-(U3-Pad9) -> GND
Routing:
- net Net-(J5-Pad3): track 0.00 -> 28.3 mm
- net Net-(C14-Pad1): track 39.2 -> 56.5 mm
- net Net-(C2-Pad1): track 17.1 -> 20.6 mm
