File: 00-produccion-pcbs/1-versiones-profes/grupo-06/g-06-perc-01-rev-a/g-06-perc-01-rev-a.kicad_sch (KiCad schematic)
At the start: 29 parts, among them J2 Barrel_Jack_Switch, J3 Barrel_Jack_Switch, J4 AudioJack2_SwitchT, SW3 SW_SPDT, U2 40106, U3 4069, U8 L7805

Commit message: añadido g06-01
Parts:
- added J5: AudioJack2_SwitchT, dis8644:PJ301M-12, symbol Connector_Audio:AudioJack2_SwitchT
Connections:
- net GND: now also U2.11, U2.13, U2.5, U2.9, U3.11, U3.13, U3.5, U3.9, J5.1
- net at C14.1, RV1.1: now also J5.2; no longer U2.1
- new net: J5.3, U2.1
- no-connect marks 24 -> 14
Other:
- moved on the sheet: C14, U2C, U2D, U2E, U2F, U3C, U3D, U3E, U3F
